File: Buttons.kicad_sch (KiCad schematic)
At the start: 40 parts

Commit message: donev1
Parts:
- removed JP1, JP10, JP11, JP12, JP13, JP14, JP15, JP16, JP17, JP18, JP19, JP2, JP20, JP3, JP4, JP5, JP6, JP7, JP8, JP9: PINHD-1X1, OF1 v1:1X01, symbol OF1 v1-eagle-import:PINHD-1X1
- removed U$1, U$10, U$11, U$12, U$13, U$14, U$15, U$16, U$17, U$18, U$19, U$2, U$20, U$3, U$4, U$5, U$6, U$7, U$8, U$9: MX-B, OF1 v1:MX-BOTH, symbol OF1 v1-eagle-import:MX-B
- added SW10, SW12, SW15, SW17, SW19, SW20, SW22, SW24, SW26, SW28, SW3, SW30, SW33, SW34, SW37, SW38, SW40, SW5, SW7, SW9: MX_SW_solder, marbastlib-mx:SW_MX_1u, symbol marbastlib-mx:MX_SW_solder
- added SW11, SW13, SW14, SW16, SW18, SW2, SW21, SW23, SW25, SW27, SW29, SW31, SW32, SW35, SW36, SW39, SW4, SW41, SW6, SW8: MX_SW_HS, marbastlib-mx:SW_MX_HS_1u, symbol marbastlib-mx:MX_SW_HS
Connections:
- net A: now also SW38.1, SW39.2
- net B: now also SW20.1, SW21.2
- net C_DN: now also SW36.2, SW37.1
- net C_LT: now also SW32.2, SW33.1
- net C_RT: now also SW40.1, SW41.2
- net C_UP: now also SW34.1, SW35.2
- net DOWN: now also SW8.2, SW9.1
- net GND: now also SW10.2, SW11.1, SW12.2, SW13.1, SW14.1, SW15.2, SW16.1, SW17.2, SW18.1, SW19.2, SW2.1, SW20.2, SW21.1, SW22.2, SW23.1, SW24.2, SW25.1, SW26.2, SW27.1, SW28.2, SW29.1, SW3.2, SW30.2, SW31.1, SW32.1, SW33.2, SW34.2, SW35.1, SW36.1, SW37.2, SW38.2, SW39.1, SW4.1, SW40.2, SW41.1, SW5.2, SW6.1, SW7.2, SW8.1, SW9.2
- net L: now also SW4.2, SW5.1
- net LEFT: now also SW6.2, SW7.1
- net LS: now also SW16.2, SW17.1
- net M1: now also SW28.1, SW29.2
- net M2: now also SW30.1, SW31.2
- net MS: now also SW18.2, SW19.1
- net R: now also SW12.1, SW13.2
- net RIGHT: now also SW10.1, SW11.2
- net START: now also SW2.2, SW3.1
- net UP: now also SW26.1, SW27.2
- net X: now also SW22.1, SW23.2
- net Y: now also SW14.2, SW15.1
- net Z: now also SW24.1, SW25.2
