File: ICOF1.kicad_pcb (KiCad board)
At the start: 2 copper layers, 347 x 156.5 mm, 96 parts, among them J1 USB C Connector, J2 JTAG_TC2030, SW1 Boot, U1 XC6206, U2 USBLC6-2SC6, U3 RP2040, U4 W25Q128JVS, Y1 12MHz

Commit message: first
Parts:
- removed J2: JTAG_TC2030, marbastlib-various:CON_TC2030_outlined
- U$1: value MX-B -> L
- moved R11 0.57 mm to (210.1, 61.4)
Routing:
- net SWD: track 24.1 -> 5.98 mm
- net SWCLK: track 24.0 -> 6.08 mm, vias 2 -> 0
- net ~{RESET}: track 10.8 -> 5.75 mm
- net XTAL_OUT: track 3.97 -> 0.00 mm
- net GND: track 50.2 -> 49.1 mm
- removed copper zone on F.Cu, net +1V1
- removed copper zone on F.Cu, net +3V3
- removed copper zone on F.Cu, net GND
Other:
- board text removed: "100nF"
- board text removed: "CHEATER"
- board text removed: "RP2040"

Commit message: donev1
Parts:
- removed R7: 10k, Resistor_SMD:R_0402_1005Metric
- D3: value GREEN -> Green_LED
- R4: footprint Resistor_SMD:R_0402_1005Metric -> Resistor_SMD:R_0603_1608Metric
- SW1: footprint Button_Switch_SMD:SW_SPST_SKQG_WithStem -> phlob2000020000:SW_TS-1187A-B-A-B
- SW10: renamed from U$5; value MX-B -> Right
- SW6: renamed from U$2; value MX-B -> Left
- SW8: renamed from U$4; value MX-B -> Down
- moved R4 0.48 mm to (220.0, 52.3)
- moved D3 0.48 mm to (223.4, 52.1), turned to 0 degrees
- moved @HOLE10 0.11 mm to (182.9, 56.0)
- renumbered U$1 to SW4
Connections:
- D3 pad 1: GND -> Net-(D3-A)
- D3 pad 2: Net-(D3-A) -> GND
- SW10 pad P$2: (no net) -> RIGHT
- SW10 pad P$3: (no net) -> RIGHT
- SW4 pad P$2: (no net) -> L
- SW4 pad P$3: (no net) -> L
- SW6 pad P$2: (no net) -> LEFT
- SW6 pad P$3: (no net) -> LEFT
- SW8 pad P$2: (no net) -> DOWN
- SW8 pad P$3: (no net) -> DOWN
- U$10 pad P$2: (no net) -> Y
- U$10 pad P$3: (no net) -> Y
- U$11 pad P$2: (no net) -> LS
- U$11 pad P$3: (no net) -> LS
- U$12 pad P$2: (no net) -> MS
- U$12 pad P$3: (no net) -> MS
- U$13 pad P$2: (no net) -> B
- U$13 pad P$3: (no net) -> B
- U$14 pad P$2: (no net) -> X
- U$14 pad P$3: (no net) -> X
- U$15 pad P$2: (no net) -> Z
- U$15 pad P$3: (no net) -> Z
- U$16 pad P$2: (no net) -> UP
- U$16 pad P$3: (no net) -> UP
- U$17 pad P$2: (no net) -> C_UP
- U$17 pad P$3: (no net) -> C_UP
- U$18 pad P$2: (no net) -> C_LT
- U$18 pad P$3: (no net) -> C_LT
- U$19 pad P$2: (no net) -> C_RT
- U$19 pad P$3: (no net) -> C_RT
- U$20 pad P$2: (no net) -> A
- U$20 pad P$3: (no net) -> A
- U$21 pad P$2: (no net) -> C_DN
- U$21 pad P$3: (no net) -> C_DN
- U$6 pad P$2: (no net) -> M1
- U$6 pad P$3: (no net) -> M1
- U$7 pad P$2: (no net) -> M2
- U$7 pad P$3: (no net) -> M2
- U$8 pad P$2: (no net) -> START
- U$8 pad P$3: (no net) -> START
- U$9 pad P$2: (no net) -> R
- U$9 pad P$3: (no net) -> R
- U3 pad 15: C_LT -> C_DN
- U3 pad 17: C_DN -> C_LT
- U3 pad 3: START -> L
- U3 pad 34: Y -> B
- U3 pad 35: B -> R
- U3 pad 36: R -> Y
- U3 pad 4: RIGHT -> LEFT
- U3 pad 6: LEFT -> RIGHT
- U3 pad 7: L -> START
Routing:
- net MS: track 7.45 -> 222.2 mm
- net LS: track 7.88 -> 218.6 mm
- net UP: track 7.80 -> 195.1 mm
- net Z: track 7.61 -> 184.7 mm
- net L: track 4.00 -> 178.1 mm
- net C_RT: track 9.64 -> 182.2 mm
- net X: track 8.26 -> 172.5 mm
- net A: track 8.64 -> 166.1 mm
- net C_DN: track 9.17 -> 151.3 mm
- net LEFT: track 4.16 -> 145.7 mm
- net M2: track 3.67 -> 132.5 mm
- net C_LT: track 7.88 -> 136.5 mm
- net Y: track 3.41 -> 127.9 mm
- net M1: track 3.83 -> 126.9 mm
- net DOWN: track 4.33 -> 117.6 mm
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- added copper zone on F.Cu, net GND
Other:
- board size 347 x 156.5 mm -> 347.1 x 156.6 mm
- board text added: "ICOF1 v1"
- board text removed: "OF1 v1"
