File: ICOF1.kicad_sch (KiCad schematic)
At the start: 46 parts, among them J1 USB C Connector, SW1 Boot, U1 XC6206, U2 USBLC6-2SC6, U3 RP2040, U4 W25Q128JVS, Y1 12MHz

Commit message: first
Parts:
- removed H1: Logo, qw-logo:qw new logo mask md, symbol Mechanical:MountingHole
- removed H10, H11, H2, H3, H4, H5, H6, H7, H8, H9: MountingHole, MountingHole:MountingHole_2.2mm_M2_ISO14580_Pad, symbol Mechanical:MountingHole
Other:
- note removed: "Mounting Holes"

Commit message: donev1
Parts:
- added D3: LED, symbol Device:LED
- added R4: R_Small, symbol Device:R_Small
Connections:
- net GND: now also D3.1 (K)
- net PICO_LED: now also R4.1
- new net: D3.2 (A), R4.2
Changed lines of the file:
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@@
+    (stroke (width 0) (type default))
+  )
+  (wire (pts (xy 205.74 125.73) (xy 210.82 125.73))
     (stroke (width 0) (type default))
   )
@@
     (stroke (width 0) (type default))
   )
+  (wire (pts (xy 226.06 125.73) (xy 228.6 125.73))
+    (stroke (width 0) (type default))
+  )
   (wire (pts (xy 146.05 176.53) (xy 148.59 176.53))
     (stroke (width 0) (type default))
@@
   )
   (wire (pts (xy 34.036 187.96) (xy 39.116 187.96))
+    (stroke (width 0) (type default))
+  )
+  (wire (pts (xy 215.9 125.73) (xy 218.44 125.73))
     (stroke (width 0) (type default))
   )
@@
     (effects (font (size 1.27 1.27)) (justify right))
     (property "Intersheetrefs" "${INTERSHEET_REFS}" (at 127.0794 58.6439 90)
+      (effects (font (size 1.27 1.27)) (justify right) hide)
+    )
+  )
+  (global_label "PICO_LED" (shape input) (at 205.74 125.73 180) (fields_autoplaced)
+    (effects (font (size 1.27 1.27)) (justify right))
+    (property "Intersheetrefs" "${INTERSHEET_REFS}" (at 193.9442 125.73 0)
       (effects (font (size 1.27 1.27)) (justify right) hide)
     )
@@
     )
   )
+  (symbol (lib_id "power:GND") (at 228.6 125.73 90) (unit 1)
+    (in_bom yes) (on_board yes) (dnp no) (fields_autoplaced)
+    (property "Reference" "#PWR034" (at 234.95 125.73 0)
+      (effects (font (size 1.27 1.27)) hide)
+    )
+    (property "Value" "GND" (at 232.41 126.365 90)
+      (effects (font (size 1.27 1.27)) (justify right))
+    )
+    (property "Footprint" "" (at 228.6 125.73 0)
+      (effects (font (size 1.27 1.27)) hide)
+    )
+    (property "Datasheet" "" (at 228.6 125.73 0)
+      (effects (font (size 1.27 1.27)) hide)
+    )
+    (pin "1")
+    (instances
+      (project "ICOF1"
+        (path "/0ee7bd02-e26d-4978-ae8c-675a718c78c0"
+          (reference "#PWR034") (unit 1)
+        )
+      )
+    )
+  )
   (symbol (lib_id "Device:C_Small") (at 143.51 181.61 270) (mirror x) (unit 1)
     (in_bom yes) (on_board yes) (dnp no)
@@
         (path "/0ee7bd02-e26d-4978-ae8c-675a718c78c0"
           (reference "R9") (unit 1)
+        )
+      )
+    )
+  )
+  (symbol (lib_id "Device:R_Small") (at 213.36 125.73 90) (unit 1)
+    (in_bom yes) (on_board yes) (dnp no) (fields_autoplaced)
+    (property "Reference" "R4" (at 213.36 120.65 90)
+      (effects (font (size 1.27 1.27)))
+    )
+    (property "Value" "R_Small" (at 213.36 123.19 90)
+      (effects (font (size 1.27 1.27)))
+    )
+    (property "Footprint" "" (at 213.36 125.73 0)
+      (effects (font (size 1.27 1.27)) hide)
+    )
+    (property "Datasheet" "~" (at 213.36 125.73 0)
+      (effects (font (size 1.27 1.27)) hide)
+    )
+    (pin "1")
+    (pin "2")
+    (instances
+      (project "ICOF1"
+        (path "/0ee7bd02-e26d-4978-ae8c-675a718c78c0"
+          (reference "R4") (unit 1)
         )
       )
@@
         )
       )
+    )
+  )
+  (symbol (lib_id "Device:LED") (at 222.25 125.73 180) (unit 1)
+    (in_bom yes) (on_board yes) (dnp no) (fields_autoplaced)
+    (property "Reference" "D3" (at 223.8375 119.38 0)
+      (effects (font (size 1.27 1.27)))
+    )
+    (property "Value" "LED" (at 223.8375 121.92 0)
+      (effects (font (size 1.27 1.27)))
+    )
+    (property "Footprint" "" (at 222.25 125.73 0)
+      (effects (font (size 1.27 1.27)) hide)
+    )
+    (property "Datasheet" "~" (at 222.25 125.73 0)
+      (effects (font (size 1.27 1.27)) hide)
+    )
+    (pin "1")
+    (pin "2")
+    (instances
+      (project "ICOF1"
+        (path "/0ee7bd02-e26d-4978-ae8c-675a718c78c0"
+          (reference "D3") (unit 1)
+        )
+      )
