File: KiCad/Buttons.kicad_sch (KiCad schematic)
At the start: 40 parts, among them SW10 MX_SW_solder, SW11 MX_SW_HS, SW12 MX_SW_solder, SW13 MX_SW_HS, SW14 MX_SW_HS, SW15 MX_SW_solder, SW16 MX_SW_HS, SW17 MX_SW_solder, SW18 MX_SW_HS, SW19 MX_SW_solder, SW2 MX_SW_HS, SW20 MX_SW_solder, SW21 MX_SW_HS, SW22 MX_SW_solder, SW23 MX_SW_HS, SW24 MX_SW_solder, SW25 MX_SW_HS, SW26 MX_SW_solder, SW27 MX_SW_HS, SW28 MX_SW_solder, SW29 MX_SW_HS, SW3 MX_SW_solder, SW30 MX_SW_solder, SW31 MX_SW_HS, SW32 MX_SW_HS, SW33 MX_SW_solder, SW34 MX_SW_solder, SW35 MX_SW_HS, SW36 MX_SW_HS, SW37 MX_SW_solder, SW38 MX_SW_solder, SW39 MX_SW_HS, SW4 MX_SW_HS, SW40 MX_SW_solder, SW41 MX_SW_HS, SW5 MX_SW_solder, SW6 MX_SW_HS, SW7 MX_SW_solder, SW8 MX_SW_HS, SW9 MX_SW_solder

Commit message: ayo!
Connections:
- net DOWN: now also SW8.1, SW9.2; no longer SW8.2, SW9.1
- net GND: now also SW8.2, SW9.1; no longer SW8.1, SW9.2
Other:
- moved on the sheet: SW8, SW9
Changed lines of the file:
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@@
     )
   )
-  (symbol (lib_id "marbastlib-mx:MX_SW_HS") (at 180.34 149.86 0) (unit 1)
-    (in_bom yes) (on_board yes) (dnp no) (fields_autoplaced)
-    (property "Reference" "SW8" (at 180.34 144.2212 0)
-      (effects (font (size 1.27 1.27)))
-    )
-    (property "Value" "MX_SW_HS" (at 180.34 145.161 0)
+  (symbol (lib_id "marbastlib-mx:MX_SW_HS") (at 180.34 149.86 180) (unit 1)
+    (in_bom yes) (on_board yes) (dnp no)
+    (property "Reference" "SW8" (at 177.8 154.94 0)
+      (effects (font (size 1.27 1.27)))
+    )
+    (property "Value" "MX_SW_HS" (at 180.34 154.559 0)
       (effects (font (size 1.27 1.27)) hide)
     )
@@
     )
   )
-  (symbol (lib_id "marbastlib-mx:MX_SW_solder") (at 180.34 149.86 180) (unit 1)
-    (in_bom yes) (on_board yes) (dnp no)
-    (property "Reference" "SW9" (at 177.3936 154.5336 0)
-      (effects (font (size 1.27 1.27)))
-    )
-    (property "Value" "MX_SW_solder" (at 180.34 155.448 0)
-      (effects (font (size 1.27 1.27)) hide)
-    )
+  (symbol (lib_id "marbastlib-mx:MX_SW_solder") (at 180.34 149.86 0) (unit 1)
+    (in_bom yes) (on_board yes) (dnp no)
+    (property "Reference" "SW9" (at 181.61 144.78 0)
+      (effects (font (size 1.27 1.27)))
+    )
+    (property "Value" "MX_SW_solder" (at 180.34 144.272 0)
+      (effects (font (size 1.27 1.27)) hide)
+    )
